Commit message: Initial commit: ROS2 workspace for thesis (excluding embedded repos)

File: install/my_sensor_description/share/my_sensor_description/urdf/lidar_camera_robot.urdf (robot description, URDF)
Before this commit: robot camera_robot, 11 links, 10 joints
Links:
- added link lidar_robot_base_link_1, mass 0.1
- added link lidar_robot_lidar_base_link_1, mass 0.1; collision cylinder length=0.1 radius=0.05; visual cylinder length=0.1 radius=0.05
- added link lidar_robot_lidar_top_link_1, mass 0.1; collision cylinder length=0.1 radius=0.05; visual cylinder length=0.1 radius=0.05
Joints:
- added joint lidar_robot_base_joint_1: type fixed, parent lidar_robot_base_link_1, child lidar_robot_lidar_base_link_1, origin xyz=0 0 0 rpy=0 0 0
- added joint lidar_robot_lidar_joint_1: type fixed, parent lidar_robot_lidar_base_link_1, child lidar_robot_lidar_top_link_1, origin xyz=0 0 0.1 rpy=0 0 0
- added joint world_to_lidar_1: type fixed, parent base_link, child lidar_robot_base_link_1, origin xyz=${lidar_1_x} ${lidar_1_y} ${lidar_1_z} rpy=${lidar_1_roll} ${lidar_1_pitch} ${lidar_1_yaw}
- joint world_to_camera: origin xyz=-7.0 -4.0 1.0 rpy=0 0 0.785 -> xyz=${camera_x} ${camera_y} ${camera_z} rpy=${camera_roll} ${camera_pitch} ${camera_yaw}
- joint world_to_camera_1: origin xyz=5.0 4.0 1.0 rpy=0 0 3.92 -> xyz=${camera_1_x} ${camera_1_y} ${camera_1_z} rpy=${camera_1_roll} ${camera_1_pitch} ${camera_1_yaw}
- joint world_to_lidar: origin xyz=0 0 1 rpy=0 0 0 -> xyz=${lidar_x} ${lidar_y} ${lidar_z} rpy=${lidar_roll} ${lidar_pitch} ${lidar_yaw}

File: src/install/my_sensor_description/share/my_sensor_description/urdf/lidar_camera_robot.urdf (robot description, URDF)
Before this commit: robot camera_robot, 11 links, 10 joints
Links:
- added link lidar_robot_base_link_1, mass 0.1
- added link lidar_robot_lidar_base_link_1, mass 0.1; collision cylinder length=0.1 radius=0.05; visual cylinder length=0.1 radius=0.05
- added link lidar_robot_lidar_top_link_1, mass 0.1; collision cylinder length=0.1 radius=0.05; visual cylinder length=0.1 radius=0.05
Joints:
- added joint lidar_robot_base_joint_1: type fixed, parent lidar_robot_base_link_1, child lidar_robot_lidar_base_link_1, origin xyz=0 0 0 rpy=0 0 0
- added joint lidar_robot_lidar_joint_1: type fixed, parent lidar_robot_lidar_base_link_1, child lidar_robot_lidar_top_link_1, origin xyz=0 0 0.1 rpy=0 0 0
- added joint world_to_lidar_1: type fixed, parent base_link, child lidar_robot_base_link_1, origin xyz=${lidar_1_x} ${lidar_1_y} ${lidar_1_z} rpy=${lidar_1_roll} ${lidar_1_pitch} ${lidar_1_yaw}
- joint world_to_camera: origin xyz=-7.0 -4.0 1.0 rpy=0 0 0.785 -> xyz=${camera_x} ${camera_y} ${camera_z} rpy=${camera_roll} ${camera_pitch} ${camera_yaw}
- joint world_to_camera_1: origin xyz=5.0 4.0 1.0 rpy=0 0 3.92 -> xyz=${camera_1_x} ${camera_1_y} ${camera_1_z} rpy=${camera_1_roll} ${camera_1_pitch} ${camera_1_yaw}
- joint world_to_lidar: origin xyz=0 0 1 rpy=0 0 0 -> xyz=${lidar_x} ${lidar_y} ${lidar_z} rpy=${lidar_roll} ${lidar_pitch} ${lidar_yaw}
